Commit message: Added move_arm script, lowered restitution coef

File: src/x6_common/x6_description/urdf/x6/x6.urdf (robot description, URDF)
Before this commit: robot x6, 10 links, 9 joints
Joints:
- joint joint5: limit lower=-1.57 upper=1.57 effort=30.0 velocity=2.617 -> lower=-1.6 upper=1.6 effort=30.0 velocity=2.617
- joint joint6: limit lower=-1.57 upper=1.57 effort=10.0 velocity=2.617 -> lower=-1.6 upper=1.6 effort=10.0 velocity=2.617
