Commit message: change color of arm so it doesnt conflict with the ball detector

File: src/kuka_kr5/kr5_description/urdf/kr.gazebo.xacro (robot description, xacro)
@@ -8,5 +8,5 @@
       </gazebo>
       <gazebo reference="link_2">
-         <material>Gazebo/Orange</material>
+         <material>Gazebo/Turquoise</material>
       </gazebo>
       <gazebo reference="link_3">
@@ -14,5 +14,5 @@
       </gazebo>
       <gazebo reference="link_4">
-         <material>Gazebo/Red</material>
+         <material>Gazebo/Turquoise</material>
       </gazebo>
       <gazebo reference="link_5">
@@ -20,5 +20,5 @@
       </gazebo>
       <gazebo reference="link_6">
-         <material>Gazebo/Yellow</material>
+         <material>Gazebo/Green</material>
       </gazebo>
       <gazebo reference="base_link">
