Commit message: Moved to TRAC-IK solver. Updated robot_controller

File: src/kuka_kr5/kr5_description/urdf/common.gazebo.xacro (robot description, xacro)
@@ -1,8 +1,6 @@
 <?xml version="1.0"?>
 <robot xmlns:xacro="http://ros.org/wiki/xacro">
-  <xacro:arg name="use_ros_control" default="False" />
+  <xacro:arg name="use_ros_control" default="false" />
   <xacro:arg name="control_period" default="0.001" />
-  <xacro:arg name="motors_controller_type" default="PositionJointInterface" /> <!-- PositionJointInterface VelocityJointInterface  EffortJointInterface-->
-  <xacro:arg name="use_the_plate" default="True" />
   <gazebo>
     <xacro:unless value="$(arg use_ros_control)">

File: src/kuka_kr5/kr5_description/urdf/kr.transmission.xacro (robot description, xacro)
@@ -35,8 +35,8 @@
       <type>transmission_interface/SimpleTransmission</type>
       <joint name="${prefix}joint_a4">
-        <hardwareInterface>hardware_interface/$(arg motors_controller_type)</hardwareInterface>
+        <hardwareInterface>hardware_interface/PositionJointInterface</hardwareInterface>
       </joint>
       <actuator name="${prefix}wrist_1_motor">
-        <hardwareInterface>hardware_interface/$(arg motors_controller_type)</hardwareInterface>
+        <hardwareInterface>hardware_interface/PositionJointInterface</hardwareInterface>
         <mechanicalReduction>1</mechanicalReduction>
       </actuator>
@@ -45,8 +45,8 @@
       <type>transmission_interface/SimpleTransmission</type>
       <joint name="${prefix}joint_a5">
-        <hardwareInterface>hardware_interface/$(arg motors_controller_type)</hardwareInterface>
+        <hardwareInterface>hardware_interface/PositionJointInterface</hardwareInterface>
       </joint>
       <actuator name="${prefix}wrist_2_motor">
-        <hardwareInterface>hardware_interface/$(arg motors_controller_type)</hardwareInterface>
+        <hardwareInterface>hardware_interface/PositionJointInterface</hardwareInterface>
         <mechanicalReduction>1</mechanicalReduction>
       </actuator>

File: src/kuka_kr5/kr5_description/urdf/kr5.urdf.xacro (robot description, xacro)
@@ -165,5 +165,5 @@
     <link name="${prefix}ee_link">
       <inertial>
-          <origin xyz="0.00983949894991115 -2.78372724487979E-05 0.17275327" rpy="0 0 0" />
+          <origin xyz="0 -.01 0.17275327" rpy="0 0 0" />
           <mass value="0.085" />
           <inertia ixx="0.002858" ixy="0" ixz="0" iyy="0.002987" iyz="0" izz="0.0001420" /> <!-- ${0.08333333333*plate_mass*plate_width}-->
@@ -240,14 +240,14 @@
     <xacro:kr_arm_gazebo prefix="${prefix}" />
     <!-- ROS base_link to UR 'Base' Coordinates transform -->
-    <link name="${prefix}base"/>
-    <joint name="${prefix}base_link-base_fixed_joint" type="fixed">
-      <!-- NOTE: this rotation is only needed as long as base_link itself is
+    <!-- NOTE: this rotation is only needed as long as base_link itself is
                  not corrected wrt the real robot (ie: rotated over 180
                  degrees)
       -->
+    <!-- <link name="${prefix}base"/>
+    <joint name="${prefix}base_link-base_fixed_joint" type="fixed">
       <origin xyz="0 0 0" rpy="0 0 ${-pi}"/>
       <parent link="${prefix}base_link"/>
       <child link="${prefix}base"/>
-    </joint>
+    </joint> -->
     <!-- Frame coincident with all-zeros TCP on UR controller -->
     <!-- <link name="${prefix}tool0"/>
