Commit message: load the world by roslaunch x6_gazebo test.launch

File: src/kuka_kr5/kr5_description/urdf/kr5.urdf.xacro (robot description, xacro)
@@ -163,5 +163,4 @@
   <!-- tool link -->
   <!-- This frame corresponds to the $FLANGE coordinate system in KUKA KRC controllers. -->
-  <xacro:if value="$(arg use_the_plate)">
      <link name="${prefix}ee_link">
         <inertial>
@@ -171,17 +170,16 @@
         </inertial>
         <visual>
-           <origin xyz="0 0 0" rpy="0 0 0" />
+           <origin xyz="0.075 0 0.27" rpy="0 3.1415 0" />
            <geometry>
-              <mesh filename="package://kr5_description/meshes/tools/plate_40.stl" scale="0.01 0.01 0.01" /> <!-- plate is 20x20x1cm if scale is 0.01 -->
+              <mesh filename="package://kr5_description/meshes/tools/paddle.stl" scale="0.001 0.001 0.001" /> <!-- plate is 20x20x1cm if scale is 0.01 -->
            </geometry>
         </visual>
         <collision>
-           <origin xyz="0 0 0" rpy="0 0 0" />
+           <origin xyz="0.075 0 0.27" rpy="0 3.1415 0" />
            <geometry>
-              <mesh filename="package://kr5_description/meshes/tools/plate_40.stl" scale="0.01 0.01 0.01" /> <!-- plate is 20x20x1 m -->
+              <mesh filename="package://kr5_description/meshes/tools/paddle.stl" scale="0.001 0.001 0.001" /> <!-- plate is 20x20x1 m -->
            </geometry>
         </collision>
      </link>
-  </xacro:if>
   <!-- joints: -->
   <joint name="${prefix}joint_a1" type="revolute">

Commit message: Fixed kuka in RVIZ and sped up simulator

File: src/kuka_kr5/kr5_description/urdf/kr5.urdf.xacro (robot description, xacro)
@@ -188,5 +188,5 @@
     <child link = "${prefix}link_1" />
     <axis xyz="0 0 1" />
-    <limit effort="150" lower="${radians(-155)}" upper="${radians(155)}" velocity="${radians(154)}" />
+    <limit effort="150" lower="${radians(-155)}" upper="${radians(155)}" velocity="${radians(15400)}" />
     <dynamics damping="0.0" friction="0.0"/>
   </joint>
@@ -196,5 +196,5 @@
       <child link = "${prefix}link_2" />
       <axis xyz="0 0 1" />
-      <limit  lower="${radians(-180)}" upper="${radians(65)}" effort="150.0" velocity="${radians(154)}"/>
+      <limit  lower="${radians(-180)}" upper="${radians(65)}" effort="150.0" velocity="${radians(15400)}"/>
       <dynamics damping="0.0" friction="0.0"/>
     </joint>
@@ -204,5 +204,5 @@
     <origin xyz="0.6 0 0" rpy="0 0 0" />
       <axis xyz="0 0 1" />
-      <limit lower="${radians(-15)}" upper="${radians(158)}"  effort="150.0" velocity="3.15"/>
+      <limit lower="${radians(-15)}" upper="${radians(158)}"  effort="150.0" velocity="315"/>
       <dynamics damping="0.0" friction="0.0"/>
     </joint>
@@ -212,5 +212,5 @@
          <origin xyz="0 -0.12 0" rpy="0 ${-pi/2} 0" />
       <axis xyz="0 0 1" />
-      <limit lower="${radians(-350)}" upper="${radians(350)}" effort="60.0" velocity="3.2"/> <!-- max should be 28 -->
+      <limit lower="${radians(-350)}" upper="${radians(350)}" effort="60.0" velocity="320"/> <!-- max should be 28 -->
       <dynamics damping="0.0" friction="0.0"/>
     </joint>
@@ -220,5 +220,5 @@
          <origin xyz="0 0 -0.62" rpy="0 ${pi/2} 0" />
       <axis xyz="0 0 1" />
-      <limit  lower="${radians(-130)}" upper="${radians(130)}" effort="60.0" velocity="3.2"/> <!-- max should be 28 -->
+      <limit  lower="${radians(-130)}" upper="${radians(130)}" effort="60.0" velocity="320"/> <!-- max should be 28 -->
       <dynamics damping="0.0" friction="0.0"/>
     </joint>
@@ -228,5 +228,5 @@
          <origin xyz="0 0 0" rpy="0 ${-pi/2} 0" />
       <axis xyz="0 0 1" />
-      <limit lower="${radians(-350)}" upper="${radians(350)}"  effort="28.0" velocity="3.2"/>
+      <limit lower="${radians(-350)}" upper="${radians(350)}"  effort="28.0" velocity="320"/>
       <dynamics damping="0.0" friction="0.0"/>
     </joint>

Commit message: update model files

File: src/kuka_kr5/kr5_description/urdf/kr5.urdf.xacro (robot description, xacro)
@@ -165,10 +165,10 @@
      <link name="${prefix}ee_link">
         <inertial>
-           <origin xyz="0.00983949894991115 -2.78372724487979E-05 -1.11022302462516E-15" rpy="0 0 0" />
-           <mass value="${plate_mass}" />
-           <inertia ixx="0.0138" ixy="0" ixz="0" iyy="0.0138" iyz="0" izz="0.0217" /> <!-- ${0.08333333333*plate_mass*plate_width}-->
+           <origin xyz="0.00983949894991115 -2.78372724487979E-05 0.17275327" rpy="0 0 0" />
+           <mass value="0.085" />
+           <inertia ixx="0.002858" ixy="0" ixz="0" iyy="0.002987" iyz="0" izz="0.0001420" /> <!-- ${0.08333333333*plate_mass*plate_width}-->
         </inertial>
         <visual>
-           <origin xyz="0.075 0 0.27" rpy="0 3.1415 0" />
+           <origin xyz="0.075 -0.012 0.253" rpy="0 3.1415 0" />
            <geometry>
               <mesh filename="package://kr5_description/meshes/tools/paddle.stl" scale="0.001 0.001 0.001" /> <!-- plate is 20x20x1cm if scale is 0.01 -->
@@ -176,5 +176,5 @@
         </visual>
         <collision>
-           <origin xyz="0.075 0 0.27" rpy="0 3.1415 0" />
+           <origin xyz="0.075 -0.012 0.253" rpy="0 3.1415 0" />
            <geometry>
               <mesh filename="package://kr5_description/meshes/tools/paddle.stl" scale="0.001 0.001 0.001" /> <!-- plate is 20x20x1 m -->

Commit message: Updated spawn_ball and fixed base_link

File: src/kuka_kr5/kr5_description/urdf/kr5.urdf.xacro (robot description, xacro)
@@ -163,32 +163,32 @@
   <!-- tool link -->
   <!-- This frame corresponds to the $FLANGE coordinate system in KUKA KRC controllers. -->
-     <link name="${prefix}ee_link">
-        <inertial>
-           <origin xyz="0.00983949894991115 -2.78372724487979E-05 0.17275327" rpy="0 0 0" />
-           <mass value="0.085" />
-           <inertia ixx="0.002858" ixy="0" ixz="0" iyy="0.002987" iyz="0" izz="0.0001420" /> <!-- ${0.08333333333*plate_mass*plate_width}-->
-        </inertial>
-        <visual>
-           <origin xyz="0.075 -0.012 0.253" rpy="0 3.1415 0" />
-           <geometry>
-              <mesh filename="package://kr5_description/meshes/tools/paddle.stl" scale="0.001 0.001 0.001" /> <!-- plate is 20x20x1cm if scale is 0.01 -->
-           </geometry>
-        </visual>
-        <collision>
-           <origin xyz="0.075 -0.012 0.253" rpy="0 3.1415 0" />
-           <geometry>
-              <mesh filename="package://kr5_description/meshes/tools/paddle.stl" scale="0.001 0.001 0.001" /> <!-- plate is 20x20x1 m -->
-           </geometry>
-        </collision>
-     </link>
-  <!-- joints: -->
-  <joint name="${prefix}joint_a1" type="revolute">
-    <origin xyz="0 0 0.4" rpy="${pi} 0 0" />
-    <parent link="${prefix}base_link" />
-    <child link = "${prefix}link_1" />
-    <axis xyz="0 0 1" />
-    <limit effort="150" lower="${radians(-155)}" upper="${radians(155)}" velocity="${radians(15400)}" />
-    <dynamics damping="0.0" friction="0.0"/>
-  </joint>
+    <link name="${prefix}ee_link">
+      <inertial>
+          <origin xyz="0.00983949894991115 -2.78372724487979E-05 0.17275327" rpy="0 0 0" />
+          <mass value="0.085" />
+          <inertia ixx="0.002858" ixy="0" ixz="0" iyy="0.002987" iyz="0" izz="0.0001420" /> <!-- ${0.08333333333*plate_mass*plate_width}-->
+      </inertial>
+      <visual>
+          <origin xyz="0.075 -0.012 0.253" rpy="0 3.1415 0" />
+          <geometry>
+            <mesh filename="package://kr5_description/meshes/tools/paddle.stl" scale="0.001 0.001 0.001" /> <!-- plate is 20x20x1cm if scale is 0.01 -->
+          </geometry>
+      </visual>
+      <collision>
+          <origin xyz="0.075 -0.012 0.253" rpy="0 3.1415 0" />
+          <geometry>
+            <mesh filename="package://kr5_description/meshes/tools/paddle.stl" scale="0.001 0.001 0.001" /> <!-- plate is 20x20x1 m -->
+          </geometry>
+      </collision>
+    </link>
+    <!-- joints: -->
+    <joint name="${prefix}joint_a1" type="revolute">
+      <origin xyz="0 0 0.4" rpy="${pi} 0 0" />
+      <parent link="${prefix}base_link" />
+      <child link = "${prefix}link_1" />
+      <axis xyz="0 0 1" />
+      <limit effort="150" lower="${radians(-155)}" upper="${radians(155)}" velocity="${radians(15400)}" />
+      <dynamics damping="0.0" friction="0.0"/>
+    </joint>
     <joint name="${prefix}joint_a2" type="revolute">
       <origin xyz="0.18 0 0" rpy="${pi/2} 0.0 0" />

File: src/kuka_kr5/kr5_description/urdf/kr5_robot.urdf.xacro (robot description, xacro)
@@ -12,5 +12,6 @@
     <parent link="world" />
     <child link = "base_link" />
-    <origin xyz="0.0 0.0 0.0" rpy="0.0 0.0 0.0" />
+    <!-- -x 0.0 -y 0.5 -z 0.762 -->
+    <origin xyz="0.0 0.5 0.762" rpy="0.0 0.0 0.0" />
   </joint>
 </robot>

Commit message: Fixed MoveIt and added planning script (#15)
* removing moveit velocity limits

* Fixed kuka in RVIZ and sped up simulator

* Added fast trajectory planning with manual time adjustment

* Adding Gazebo paths to package.xml

* Updated spawn_ball and fixed base_link

File: src/kuka_kr5/kr5_description/urdf/kr5.urdf.xacro (robot description, xacro)
@@ -163,32 +163,32 @@
   <!-- tool link -->
   <!-- This frame corresponds to the $FLANGE coordinate system in KUKA KRC controllers. -->
-     <link name="${prefix}ee_link">
-        <inertial>
-           <origin xyz="0.00983949894991115 -2.78372724487979E-05 0.17275327" rpy="0 0 0" />
-           <mass value="0.085" />
-           <inertia ixx="0.002858" ixy="0" ixz="0" iyy="0.002987" iyz="0" izz="0.0001420" /> <!-- ${0.08333333333*plate_mass*plate_width}-->
-        </inertial>
-        <visual>
-           <origin xyz="0.075 -0.012 0.253" rpy="0 3.1415 0" />
-           <geometry>
-              <mesh filename="package://kr5_description/meshes/tools/paddle.stl" scale="0.001 0.001 0.001" /> <!-- plate is 20x20x1cm if scale is 0.01 -->
-           </geometry>
-        </visual>
-        <collision>
-           <origin xyz="0.075 -0.012 0.253" rpy="0 3.1415 0" />
-           <geometry>
-              <mesh filename="package://kr5_description/meshes/tools/paddle.stl" scale="0.001 0.001 0.001" /> <!-- plate is 20x20x1 m -->
-           </geometry>
-        </collision>
-     </link>
-  <!-- joints: -->
-  <joint name="${prefix}joint_a1" type="revolute">
-    <origin xyz="0 0 0.4" rpy="${pi} 0 0" />
-    <parent link="${prefix}base_link" />
-    <child link = "${prefix}link_1" />
-    <axis xyz="0 0 1" />
-    <limit effort="150" lower="${radians(-155)}" upper="${radians(155)}" velocity="${radians(154)}" />
-    <dynamics damping="0.0" friction="0.0"/>
-  </joint>
+    <link name="${prefix}ee_link">
+      <inertial>
+          <origin xyz="0.00983949894991115 -2.78372724487979E-05 0.17275327" rpy="0 0 0" />
+          <mass value="0.085" />
+          <inertia ixx="0.002858" ixy="0" ixz="0" iyy="0.002987" iyz="0" izz="0.0001420" /> <!-- ${0.08333333333*plate_mass*plate_width}-->
+      </inertial>
+      <visual>
+          <origin xyz="0.075 -0.012 0.253" rpy="0 3.1415 0" />
+          <geometry>
+            <mesh filename="package://kr5_description/meshes/tools/paddle.stl" scale="0.001 0.001 0.001" /> <!-- plate is 20x20x1cm if scale is 0.01 -->
+          </geometry>
+      </visual>
+      <collision>
+          <origin xyz="0.075 -0.012 0.253" rpy="0 3.1415 0" />
+          <geometry>
+            <mesh filename="package://kr5_description/meshes/tools/paddle.stl" scale="0.001 0.001 0.001" /> <!-- plate is 20x20x1 m -->
+          </geometry>
+      </collision>
+    </link>
+    <!-- joints: -->
+    <joint name="${prefix}joint_a1" type="revolute">
+      <origin xyz="0 0 0.4" rpy="${pi} 0 0" />
+      <parent link="${prefix}base_link" />
+      <child link = "${prefix}link_1" />
+      <axis xyz="0 0 1" />
+      <limit effort="150" lower="${radians(-155)}" upper="${radians(155)}" velocity="${radians(15400)}" />
+      <dynamics damping="0.0" friction="0.0"/>
+    </joint>
     <joint name="${prefix}joint_a2" type="revolute">
       <origin xyz="0.18 0 0" rpy="${pi/2} 0.0 0" />
@@ -196,5 +196,5 @@
       <child link = "${prefix}link_2" />
       <axis xyz="0 0 1" />
-      <limit  lower="${radians(-180)}" upper="${radians(65)}" effort="150.0" velocity="${radians(154)}"/>
+      <limit  lower="${radians(-180)}" upper="${radians(65)}" effort="150.0" velocity="${radians(15400)}"/>
       <dynamics damping="0.0" friction="0.0"/>
     </joint>
@@ -204,5 +204,5 @@
     <origin xyz="0.6 0 0" rpy="0 0 0" />
       <axis xyz="0 0 1" />
-      <limit lower="${radians(-15)}" upper="${radians(158)}"  effort="150.0" velocity="3.15"/>
+      <limit lower="${radians(-15)}" upper="${radians(158)}"  effort="150.0" velocity="315"/>
       <dynamics damping="0.0" friction="0.0"/>
     </joint>
@@ -212,5 +212,5 @@
          <origin xyz="0 -0.12 0" rpy="0 ${-pi/2} 0" />
       <axis xyz="0 0 1" />
-      <limit lower="${radians(-350)}" upper="${radians(350)}" effort="60.0" velocity="3.2"/> <!-- max should be 28 -->
+      <limit lower="${radians(-350)}" upper="${radians(350)}" effort="60.0" velocity="320"/> <!-- max should be 28 -->
       <dynamics damping="0.0" friction="0.0"/>
     </joint>
@@ -220,5 +220,5 @@
          <origin xyz="0 0 -0.62" rpy="0 ${pi/2} 0" />
       <axis xyz="0 0 1" />
-      <limit  lower="${radians(-130)}" upper="${radians(130)}" effort="60.0" velocity="3.2"/> <!-- max should be 28 -->
+      <limit  lower="${radians(-130)}" upper="${radians(130)}" effort="60.0" velocity="320"/> <!-- max should be 28 -->
       <dynamics damping="0.0" friction="0.0"/>
     </joint>
@@ -228,5 +228,5 @@
          <origin xyz="0 0 0" rpy="0 ${-pi/2} 0" />
       <axis xyz="0 0 1" />
-      <limit lower="${radians(-350)}" upper="${radians(350)}"  effort="28.0" velocity="3.2"/>
+      <limit lower="${radians(-350)}" upper="${radians(350)}"  effort="28.0" velocity="320"/>
       <dynamics damping="0.0" friction="0.0"/>
     </joint>

Commit message: Fixed tool frame planning. Fixed table height. Ran MoveIt setup assistant for new files

File: src/kuka_kr5/kr5_description/urdf/kr5.urdf.xacro (robot description, xacro)
@@ -170,5 +170,5 @@
       </inertial>
       <visual>
-          <origin xyz="0.075 -0.012 0.253" rpy="0 3.1415 0" />
+          <origin xyz="0.075 -0.012 0.06" rpy="0 ${pi} 0" />
           <geometry>
             <mesh filename="package://kr5_description/meshes/tools/paddle.stl" scale="0.001 0.001 0.001" /> <!-- plate is 20x20x1cm if scale is 0.01 -->
@@ -176,5 +176,5 @@
       </visual>
       <collision>
-          <origin xyz="0.075 -0.012 0.253" rpy="0 3.1415 0" />
+          <origin xyz="0.075 -0.012 0.06" rpy="0 ${pi} 0" />
           <geometry>
             <mesh filename="package://kr5_description/meshes/tools/paddle.stl" scale="0.001 0.001 0.001" /> <!-- plate is 20x20x1 m -->
@@ -234,6 +234,7 @@
       <parent link="${prefix}link_6" />
       <child link = "${prefix}ee_link" />
-      <origin xyz="0 0 -0.115" rpy="0 ${-pi} ${-pi/2}" />
-    </joint>
+      <origin xyz="0 0 -.308" rpy="0 ${-pi} ${-pi/2}" />
+    </joint>
+<!-- -.368 is 0 visual offset -->
     <xacro:kr_arm_transmission prefix="${prefix}" />
     <xacro:kr_arm_gazebo prefix="${prefix}" />
@@ -250,10 +251,10 @@
     </joint>
     <!-- Frame coincident with all-zeros TCP on UR controller -->
-    <link name="${prefix}tool0"/>
+    <!-- <link name="${prefix}tool0"/>
     <joint name="${prefix}wrist_3_link-tool0_fixed_joint" type="fixed">
       <origin xyz="0 0.115 0" rpy="${pi/-2.0} 0 0"/>
       <parent link="${prefix}link_6"/>
       <child link="${prefix}tool0"/>
-    </joint>
+    </joint> -->
   </xacro:macro>
 </robot>

Commit message: play with the values of dist and controller_hit in ball_prediction.py

File: src/kuka_kr5/kr5_description/urdf/kr5.urdf.xacro (robot description, xacro)
@@ -180,6 +180,19 @@
             <mesh filename="package://kr5_description/meshes/tools/paddle.stl" scale="0.001 0.001 0.001" /> <!-- plate is 20x20x1 m -->
           </geometry>
-      </collision>
-    </link>
+          <surface>
+            <bounce restitution_coefficient="0.1" threshold="0.01"/>
+          </surface>
+      </collision>
+    </link>
+    <gazebo reference="${prefix}ee_link">
+      <mu1 value="100.0" />
+      <mu2 value="0.1" />
+      <maxVel value="10.0"/>
+      <kp value="1000.0" />
+      <kd value="1.0" />
+      <fdir1 value="1 0 0" />
+      <material>Gazebo/Grey</material>
+      <turnGravityOff>false</turnGravityOff>
+    </gazebo>
     <!-- joints: -->
     <joint name="${prefix}joint_a1" type="revolute">
